Commit message: bug fix and add gates environment

File: PyFlyt/models/race_gate.urdf (robot description, URDF)
Before this commit: robot cube, 4 links, 3 joints
Links:
- added link bottom_link, mass 1; collision box size=0.05 0.5 0.05; visual box size=0.05 0.5 0.05
- link base_link: geometry visual box size=0 0 0
- link left_link: geometry collision box size=0.05 0.05 0.4; visual box size=0.05 0.05 0.4
- link right_link: geometry collision box size=0.05 0.05 0.4; visual box size=0.05 0.05 0.4
- link top_link: geometry collision box size=0.05 0.5 0.05; visual box size=0.05 0.5 0.05
Joints:
- added joint base_to_bottom: type fixed, parent base_link, child bottom_link, origin xyz=0.0 0.0 -0.225
- joint base_to_left: origin xyz=-0.175 0.0 0.175 -> xyz=0.0 -0.225 0.0
- joint base_to_right: origin xyz=0.175 0.0 0.175 -> xyz=0.0 0.225 0.0
- joint base_to_top: origin xyz=0.0 0.0 0.35 -> xyz=0.0 0.0 0.225

File: PyFlyt/models/target.urdf (robot description, URDF)
Before this commit: robot cube, 1 links, 0 joints
Links:
- link base_link: geometry visual sphere radius=0.05

File: PyFlyt/models/vehicles/cf2x.urdf (robot description, URDF)
Before this commit: robot cf2, 6 links, 5 joints
Links:
- link base_link: geometry collision box size=0.09 0.09 0.02; visual mesh filename=./cf2.dae scale=1 1 1
