Commit message: update some params and add reward for pole uprightness

File: PyFlyt/models/pole.urdf (robot description, URDF)
Before this commit: robot cube, 2 links, 1 joints
Links:
- link base_link: geometry visual box size=0 0 0; visual sphere radius=0.01

Commit message: stashing

File: PyFlyt/models/pole.urdf (robot description, URDF)
Before this commit: robot cube, 2 links, 1 joints
Links:
- added link bottom_link, mass 0.0; collision sphere length=1.0 radius=0.01; visual sphere length=1.0 radius=0.01
- link base_link: mass 0.001 -> 0.01
Joints:
- added joint base_to_bottom: type fixed, parent base_link, child bottom_link, origin xyz=0.0 0.0 -1.0

Commit message: np concat and ther things

File: PyFlyt/models/pole.urdf (robot description, URDF)
Before this commit: robot cube, 3 links, 2 joints
Links:
- removed link pole_link
- added link top_link, mass 0.0; visual box size=0 0 0; visual sphere radius=0.04
- link base_link: mass 0.01 -> 0.2; geometry collision cylinder length=1.0 radius=0.005; visual cylinder length=1.0 radius=0.005
- link bottom_link: geometry visual box size=0 0 0; visual sphere radius=0.01
Joints:
- removed joint base_to_pole
- added joint base_to_top: type fixed, parent base_link, child top_link, origin xyz=0.0 0.0 0.5
- joint base_to_bottom: origin xyz=0.0 0.0 -1.0 -> xyz=0.0 0.0 -0.5
