Commit message: smaller ball and rew for staying at center

File: PyFlyt/models/ball_and_string.urdf (robot description, URDF)
Before this commit: robot ball_and_string, 2 links, 1 joints
Links:
- link ball: geometry collision sphere radius=0.05; visual sphere radius=0.05

Commit message: longer string

File: PyFlyt/models/ball_and_string.urdf (robot description, URDF)
Before this commit: robot ball_and_string, 2 links, 1 joints
Joints:
- joint ball_to_base: limit lower=0.0 upper=0.4 effort=0.0 -> lower=0.0 upper=1.0 effort=0.0; origin xyz=0 0 0.3 rpy=0 0 0 -> xyz=0 0 0.5 rpy=0 0 0

Commit message: allow negative string length

File: PyFlyt/models/ball_and_string.urdf (robot description, URDF)
Before this commit: robot ball_and_string, 2 links, 1 joints
Joints:
- joint ball_to_base: limit lower=0.0 upper=1.0 effort=0.0 -> lower=-0.5 upper=1.0 effort=0.0
