Commit message: add back penalty for aggressive maneuvres

File: PyFlyt/models/cup.urdf (robot description, URDF)
Before this commit: robot cup, 5 links, 4 joints
Links:
- link back_wall: geometry collision box size=0.2 0.01 0.1; visual box size=0.2 0.01 0.1
- link front_wall: geometry collision box size=0.2 0.01 0.1; visual box size=0.2 0.01 0.1
- link left_wall: geometry collision box size=0.01 0.2 0.1; visual box size=0.01 0.2 0.1
- link right_wall: geometry collision box size=0.01 0.2 0.1; visual box size=0.01 0.2 0.1
Joints:
- joint base_to_back: origin xyz=0.0 0.075 0.05 -> xyz=0.0 0.1 0.05
- joint base_to_front: origin xyz=0.0 -0.075 0.05 -> xyz=0.0 -0.1 0.05
- joint base_to_left: origin xyz=0.075 0.0 0.05 -> xyz=0.1 0.0 0.05
- joint base_to_right: origin xyz=-0.075 0.0 0.05 -> xyz=-0.1 0.0 0.05
