Commit message: minor update to gymnasium among other things

File: PyFlyt/models/vehicles/cf2x.urdf (robot description, URDF)
Before this commit: robot cf2, 6 links, 5 joints
Links:
- removed link prop0_link
- added link prop4_link, mass 0
Joints:
- removed joint prop0_joint
- added joint prop4_joint: type fixed, parent base_link, child prop4_link
