Commit message: 1st implementation

File: PyFlyt/models/vehicles/fixedwing/fixedwing.urdf (robot description, URDF)
Before this commit: robot FW_UAV, 6 links, 5 joints
Links:
- removed link center_of_mass_link
- removed link prop1_link
- removed link prop2_link
- removed link prop3_link
- removed link prop4_link
- added link ail_left_link, mass 0.1; collision box size=0.3 0.3 0.1
- added link ail_right_link, mass 0.1; collision box size=0.3 0.3 0.1
- added link fuselage_link, mass 1; collision box size=0.2 1.4 0.2
- added link horizontal_tail_link, mass 0.1; collision box size=0.6 0.3 0.1
- added link main_wing_link, mass 0.5; collision box size=1.8 0.3 0.1
- added link motor_link, mass 0
- added link vertical_tail_link, mass 0.05; collision box size=0.1 0.3 0.3
- link base_link: mass 0.027 -> 0.3; geometry collision box size=0.2 0.1 0.2
Joints:
- removed joint center_of_mass_joint
- removed joint prop1_joint
- removed joint prop2_joint
- removed joint prop3_joint
- removed joint prop4_joint
- added joint ail_left_joint: type fixed, parent base_link, child ail_left_link, origin xyz=-0.95 -0.5 0 rpy=0 0 0
- added joint ail_right_joint: type fixed, parent base_link, child ail_right_link, origin xyz=0.95 -0.5  0 rpy=0 0 0
- added joint fuselage_joint: type fixed, parent base_link, child fuselage_link, origin xyz=0 -0.8 0 rpy=0 0 0
- added joint horizontal_tail_joint: type fixed, parent base_link, child horizontal_tail_link, origin xyz=0 -1.1 0 rpy=0 0 0
- added joint main_wing_joint: type fixed, parent base_link, child main_wing_link, origin xyz=0 -0.5 0 rpy=0 0 0
- added joint motor_joint: type fixed, parent base_link, child motor_link, origin xyz=0 0 0 rpy=0 0 0
- added joint vertical_tail_joint: type fixed, parent base_link, child vertical_tail_link, origin xyz=0 -1.1 0.15 rpy=0 0 0

Commit message: First working fixed wing UAV controllable with DS4

File: PyFlyt/models/vehicles/fixedwing/fixedwing.urdf (robot description, URDF)
Before this commit: robot fixedwing, 8 links, 7 joints
Joints:
- joint fuselage_joint: origin xyz=0 -0.8 0 rpy=0 0 0 -> xyz=0 -0.5 0 rpy=0 0 0

Commit message: Allow spawn initial velocity

File: PyFlyt/models/vehicles/fixedwing/fixedwing.urdf (robot description, URDF)
Before this commit: robot fixedwing, 8 links, 7 joints
Joints:
- joint fuselage_joint: origin xyz=0 -0.5 0 rpy=0 0 0 -> xyz=0 -0.45 0 rpy=0 0 0

Commit message: Commited fixed wing UAV, included FWTargets env

File: PyFlyt/models/vehicles/fixedwing/fixedwing.urdf (robot description, URDF)
Before this commit: robot fixedwing, 8 links, 7 joints
Links:
- link ail_left_link: mass 0.1 -> 0.2
- link ail_right_link: mass 0.1 -> 0.2

Commit message: fix fixedwing and rocket axis conventions

File: PyFlyt/models/vehicles/fixedwing/fixedwing.urdf (robot description, URDF)
Before this commit: robot fixedwing, 8 links, 7 joints
Links:
- link base_link: geometry collision box size=0.1 0.2 0.2
- link fuselage_link: geometry collision box size=1.4 0.2 0.2
- link horizontal_tail_link: geometry collision box size=0.3 0.6 0.1
- link main_wing_link: geometry collision box size=0.3 1.8 0.1
- link vertical_tail_link: geometry collision box size=0.3 0.1 0.3
Joints:
- joint ail_left_joint: origin xyz=-0.95 -0.5 0 rpy=0 0 0 -> xyz=-0.5 0.95 0 rpy=0 0 0
- joint ail_right_joint: origin xyz=0.95 -0.5  0 rpy=0 0 0 -> xyz=-0.5 -0.95  0 rpy=0 0 0
- joint fuselage_joint: origin xyz=0 -0.45 0 rpy=0 0 0 -> xyz=-0.45 0 0 rpy=0 0 0
- joint horizontal_tail_joint: origin xyz=0 -1.1 0 rpy=0 0 0 -> xyz=-1.1 0 0 rpy=0 0 0
- joint main_wing_joint: origin xyz=0 -0.5 0 rpy=0 0 0 -> xyz=-0.5 0 0 rpy=0 0 0
- joint vertical_tail_joint: origin xyz=0 -1.1 0.15 rpy=0 0 0 -> xyz=-1.1 0 0.15 rpy=0 0 0

File: PyFlyt/models/vehicles/rocket/rocket.urdf (robot description, URDF)
Before this commit: robot rocket, 10 links, 9 joints
Links:
- removed link fin_neg_z
- removed link fin_pos_z
- added link fin_neg_x, mass 0.05; collision box size=0.3 0.03 0.3
- added link fin_pos_x, mass 0.05; collision box size=0.3 0.03 0.3
- link fin_neg_y: geometry collision box size=0.03 0.3 0.3
- link fin_pos_y: geometry collision box size=0.03 0.3 0.3
- link leg_1: geometry collision box size=0.05 0.5 0.05
- link leg_2: geometry collision box size=0.05 0.5 0.05
- link leg_3: geometry collision box size=0.05 0.5 0.05
Joints:
- removed joint fin_neg_z_joint
- removed joint fin_pos_z_joint
- added joint fin_neg_x_joint: type fixed, parent base_link, child fin_neg_x, origin xyz=-0.35 0 2.051 rpy=0 0 0
- added joint fin_pos_x_joint: type fixed, parent base_link, child fin_pos_x, origin xyz=0.35 0 2.051 rpy=0 0 0
- joint booster_joint: origin xyz=0 -2 0 rpy=0 0 0 -> xyz=0 0 -2 rpy=0 0 0
- joint fin_neg_y_joint: origin xyz=-0.35 2.051 0 rpy=0 0 0 -> xyz=0 -0.35 2.051 rpy=0 0 0
- joint fin_pos_y_joint: origin xyz=0.35 2.051 0 rpy=0 0 0 -> xyz=0 0.35 2.051 rpy=0 0 0
- joint leg_1_joint: origin xyz=0.0 -2.4 0.35 rpy=0 0 0 -> xyz=0.0 0.35 -2.4 rpy=0 0 0
- joint leg_2_joint: origin xyz=-0.3031 -2.4 -0.175 rpy=0 4.188 0 -> xyz=0.3031 -0.175 -2.4 rpy=0 0 4.188
- joint leg_3_joint: origin xyz=0.3031 -2.4 -0.175 rpy=0 -4.188 0 -> xyz=-0.3031 -0.175 -2.4 rpy=0 0 -4.188

Commit message: fix geometry of primi drone for now, no control laws yet

File: PyFlyt/models/vehicles/fixedwing/fixedwing.urdf (robot description, URDF)
Before this commit: robot fixedwing, 8 links, 7 joints
Links:
- link ail_left_link: geometry collision box size=0.31 0.3 0.06; visual box size=0.31 0.3 0.06
- link ail_right_link: geometry collision box size=0.31 0.3 0.06; visual box size=0.31 0.3 0.06
- link base_link: geometry 
- link fuselage_link: geometry collision box size=1.4 0.2 0.2; visual box size=1.4 0.2 0.2
- link horizontal_tail_link: geometry collision box size=0.3 0.6 0.05; visual box size=0.3 0.6 0.05
- link main_wing_link: geometry collision box size=0.3 1.8 0.05; visual box size=0.3 1.8 0.05
- link vertical_tail_link: geometry collision box size=0.3 0.05 0.3; visual box size=0.3 0.05 0.3

File: PyFlyt/models/vehicles/primitive_drone/primitive_drone.urdf (robot description, URDF)
Before this commit: robot drone, 5 links, 4 joints
Links:
- link back_left_prop: mass 0.05 -> 0; geometry collision cylinder length=0.01 radius=0.01; visual cylinder length=0.01 radius=0.12
- link back_right_prop: mass 0.05 -> 0; geometry collision cylinder length=0.01 radius=0.01; visual cylinder length=0.01 radius=0.12
- link base_link: mass 0.5 -> 1.0; geometry collision box size=0.15 0.1 0.05; visual box size=0.2 0.1 0.05
- link front_left_prop: mass 0.05 -> 0; geometry collision cylinder length=0.01 radius=0.01; visual cylinder length=0.01 radius=0.12
- link front_right_prop: mass 0.05 -> 0; geometry collision cylinder length=0.01 radius=0.01; visual cylinder length=0.01 radius=0.12
Joints:
- joint base_to_back_left_prop: origin xyz=-0.25 0.25 0.060000000000000005 -> xyz=-0.16 0.16 0
- joint base_to_back_right_prop: origin xyz=-0.25 -0.25 0.060000000000000005 -> xyz=-0.16 -0.16 0
- joint base_to_front_left_prop: origin xyz=0.25 0.25 0.060000000000000005 -> xyz=0.16 0.16 0
- joint base_to_front_right_prop: origin xyz=0.25 -0.25 0.060000000000000005 -> xyz=0.16 -0.16 0

File: PyFlyt/models/vehicles/rocket/rocket.urdf (robot description, URDF)
Before this commit: robot rocket, 10 links, 9 joints
Links:
- link base_link: geometry collision cylinder length=4.77 radius=0.185; visual cylinder length=4.77 radius=0.185
- link booster_link: geometry collision cylinder length=0.5 radius=0.25; visual cylinder length=0.5 radius=0.25
- link fin_neg_x: geometry collision box size=0.3 0.03 0.3; visual box size=0.3 0.03 0.3
- link fin_neg_y: geometry collision box size=0.03 0.3 0.3; visual box size=0.03 0.3 0.3
- link fin_pos_x: geometry collision box size=0.3 0.03 0.3; visual box size=0.3 0.03 0.3
- link fin_pos_y: geometry collision box size=0.03 0.3 0.3; visual box size=0.03 0.3 0.3
- link leg_1: geometry collision box size=0.05 0.5 0.05; visual box size=0.05 0.5 0.05
- link leg_2: geometry collision box size=0.05 0.5 0.05; visual box size=0.05 0.5 0.05
- link leg_3: geometry collision box size=0.05 0.5 0.05; visual box size=0.05 0.5 0.05
