Commit message: update primitive drone

File: PyFlyt/models/vehicles/primitive_drone/primitive_drone.urdf (robot description, URDF)
Before this commit: robot car, 6 links, 5 joints
Links:
- removed link back_left_wheel
- removed link back_right_wheel
- removed link camera
- removed link front_left_wheel
- removed link front_right_wheel
- added link back_left_prop, mass 0.05; collision cylinder length=0.01 radius=0.01; visual cylinder length=0.01 radius=0.2
- added link back_right_prop, mass 0.05; collision cylinder length=0.01 radius=0.01; visual cylinder length=0.01 radius=0.2
- added link front_left_prop, mass 0.05; collision cylinder length=0.01 radius=0.01; visual cylinder length=0.01 radius=0.2
- added link front_right_prop, mass 0.05; collision cylinder length=0.01 radius=0.01; visual cylinder length=0.01 radius=0.2
- link base_link: mass 0.05 -> 0.5; geometry collision box size=0.4 0.2 0.1; visual box size=0.4 0.2 0.1
Joints:
- removed joint base_to_back_left_wheel
- removed joint base_to_back_right_wheel
- removed joint base_to_camera
- removed joint base_to_front_left_wheel
- removed joint base_to_front_right_wheel
- added joint base_to_back_left_prop: type fixed, parent base_link, child back_left_prop, origin xyz=-0.25 0.25 0.060000000000000005, axis 1 0 0
- added joint base_to_back_right_prop: type fixed, parent base_link, child back_right_prop, origin xyz=-0.25 -0.25 0.060000000000000005, axis 1 0 0
- added joint base_to_front_left_prop: type fixed, parent base_link, child front_left_prop, origin xyz=0.25 0.25 0.060000000000000005, axis 1 0 0
- added joint base_to_front_right_prop: type fixed, parent base_link, child front_right_prop, origin xyz=0.25 -0.25 0.060000000000000005, axis 1 0 0

Commit message: add primitive drone

File: PyFlyt/models/vehicles/primitive_drone/primitive_drone.urdf (robot description, URDF)
Before this commit: robot drone, 5 links, 4 joints
Links:
- link back_left_prop: geometry collision cylinder length=0.01 radius=0.12; visual cylinder length=0.01 radius=0.12
- link back_right_prop: geometry collision cylinder length=0.01 radius=0.12; visual cylinder length=0.01 radius=0.12
- link base_link: geometry collision box size=0.2 0.1 0.05; visual box size=0.2 0.1 0.05
- link front_left_prop: geometry collision cylinder length=0.01 radius=0.12; visual cylinder length=0.01 radius=0.12
- link front_right_prop: geometry collision cylinder length=0.01 radius=0.12; visual cylinder length=0.01 radius=0.12
