Commit message: fix bug in lifting surface and flesh out rocket more

File: PyFlyt/models/vehicles/rocket/rocket.urdf (robot description, URDF)
Before this commit: robot rocket, 9 links, 8 joints
Links:
- removed link fin_neg_y
- removed link fin_pos_y
Joints:
- removed joint fin_neg_y_joint
- removed joint fin_pos_y_joint

Commit message: fix rocket

File: PyFlyt/models/vehicles/rocket/rocket.urdf (robot description, URDF)
Before this commit: robot rocket, 7 links, 6 joints
Links:
- added link fin_neg_z, mass 0.05; collision box size=0.03 0.3 0.3
- added link fin_pos_z, mass 0.05; collision box size=0.03 0.3 0.3
- added link payload_link, mass 0.3; collision sphere radius=0.2
- link fin_neg_x: geometry collision box size=0.3 0.3 0.03
- link fin_pos_x: geometry collision box size=0.3 0.3 0.03
- link leg_1: geometry collision box size=0.05 0.05 0.5
- link leg_2: geometry collision box size=0.05 0.05 0.5
- link leg_3: geometry collision box size=0.05 0.05 0.5
Joints:
- added joint fin_neg_y_joint: type fixed, parent base_link, child fin_neg_z, origin xyz=0 2.35 -0.35 rpy=0 0 0
- added joint fin_pos_y_joint: type fixed, parent base_link, child fin_pos_z, origin xyz=0 2.35 0.35 rpy=0 0 0
- added joint payload_joint: type fixed, parent base_link, child payload_link, origin xyz=0 2.5 0 rpy=0 0 0
- joint booster_joint: origin xyz=0 0 -2.5 rpy=0 0 0 -> xyz=0 -2.5 0 rpy=0 0 0
- joint fin_neg_x_joint: origin xyz=-0.35 0 2.35 rpy=0 0 0 -> xyz=-0.35 2.35 0 rpy=0 0 0
- joint fin_pos_x_joint: origin xyz=0.35 0 2.35 rpy=0 0 0 -> xyz=0.35 2.35 0 rpy=0 0 0
- joint leg_1_joint: origin xyz=0.35 0 -2.35 rpy=0 1.0 0 -> xyz=0.0 -2.7 0.35 rpy=0 0 0
- joint leg_2_joint: origin xyz=-0.175 0.3031 -2.35 rpy=0 1.0 2.0944 -> xyz=-0.3031 -2.7 -0.175 rpy=0 4.188 0
- joint leg_3_joint: origin xyz=-0.175 -0.3031 -2.35 rpy=0 1.0 4.1887 -> xyz=0.3031 -2.7 -0.175 rpy=0 -4.188 0

Commit message: semi completed rocket model

File: PyFlyt/models/vehicles/rocket/rocket.urdf (robot description, URDF)
Before this commit: robot rocket, 10 links, 9 joints
Links:
- removed link payload_link
- added link fueltank_link, mass 410.9; collision cylinder length=1 radius=0.1
- link base_link: mass 1.0 -> 138.0; geometry collision cylinder length=4.77 radius=0.185
- link booster_link: mass 0.3 -> 0.0; geometry collision cylinder length=0.5 radius=0.25
Joints:
- removed joint payload_joint
- added joint fueltank_joint: type fixed, parent base_link, child fueltank_link, origin xyz=0 0 0 rpy=0 0 0
- joint booster_joint: origin xyz=0 -2.5 0 rpy=0 0 0 -> xyz=0 -2 0 rpy=0 0 0
- joint fin_neg_x_joint: origin xyz=-0.35 2.35 0 rpy=0 0 0 -> xyz=-0.35 2.051 0 rpy=0 0 0
- joint fin_neg_y_joint: origin xyz=0 2.35 -0.35 rpy=0 0 0 -> xyz=0 2.051 -0.35 rpy=0 0 0
- joint fin_pos_x_joint: origin xyz=0.35 2.35 0 rpy=0 0 0 -> xyz=0.35 2.051 0 rpy=0 0 0
- joint fin_pos_y_joint: origin xyz=0 2.35 0.35 rpy=0 0 0 -> xyz=0 2.051 0.35 rpy=0 0 0
- joint leg_1_joint: origin xyz=0.0 -2.7 0.35 rpy=0 0 0 -> xyz=0.0 -2.4 0.35 rpy=0 0 0
- joint leg_2_joint: origin xyz=-0.3031 -2.7 -0.175 rpy=0 4.188 0 -> xyz=-0.3031 -2.4 -0.175 rpy=0 4.188 0
- joint leg_3_joint: origin xyz=0.3031 -2.7 -0.175 rpy=0 -4.188 0 -> xyz=0.3031 -2.4 -0.175 rpy=0 -4.188 0

Commit message: major refactor

File: PyFlyt/models/vehicles/rocket/rocket.urdf (robot description, URDF)
Before this commit: robot rocket, 10 links, 9 joints
Links:
- removed link fin_neg_x
- removed link fin_pos_x
- added link fin_neg_y, mass 0.05; collision box size=0.3 0.3 0.03
- added link fin_pos_y, mass 0.05; collision box size=0.3 0.3 0.03
Joints:
- removed joint fin_neg_x_joint
- removed joint fin_pos_x_joint
- added joint fin_neg_z_joint: type fixed, parent base_link, child fin_neg_z, origin xyz=0 2.051 -0.35 rpy=0 0 0
- added joint fin_pos_z_joint: type fixed, parent base_link, child fin_pos_z, origin xyz=0 2.051 0.35 rpy=0 0 0
- joint fin_neg_y_joint: child fin_neg_z -> fin_neg_y; origin xyz=0 2.051 -0.35 rpy=0 0 0 -> xyz=-0.35 2.051 0 rpy=0 0 0
- joint fin_pos_y_joint: child fin_pos_z -> fin_pos_y; origin xyz=0 2.051 0.35 rpy=0 0 0 -> xyz=0.35 2.051 0 rpy=0 0 0

Commit message: update rocket model

File: PyFlyt/models/vehicles/rocket/rocket.urdf (robot description, URDF)
Before this commit: robot rocket, 10 links, 9 joints
Links:
- link base_link: mass 138.0 -> 69.0
- link booster_link: mass 0.0 -> 69.0

Commit message: fix rocket inertia properties

File: PyFlyt/models/vehicles/rocket/rocket.urdf (robot description, URDF)
Before this commit: robot rocket, 10 links, 9 joints
Links:
- link base_link: mass 69.0 -> 91.0
- link booster_link: mass 69.0 -> 47
