Commit message: update quadx normal area

File: PyFlyt/models/vehicles/cf2x/cf2x.urdf (robot description, URDF)
Before this commit: robot cf2, 6 links, 5 joints
Links:
- added link body, mass 0
Joints:
- added joint body_link: type fixed, parent base_link, child body, origin xyz=0 0 0, axis 0 0 0

File: PyFlyt/models/vehicles/primitive_drone/primitive_drone.urdf (robot description, URDF)
Before this commit: robot drone, 5 links, 4 joints
Links:
- added link body, mass 0
Joints:
- added joint body_link: type fixed, parent base_link, child body, origin xyz=0 0 0, axis 0 0 0
