Commit message: remove need for three separate wings

File: PyFlyt/models/vehicles/acrowing/acrowing.urdf (robot description, URDF)
Before this commit: robot acrowing, 9 links, 8 joints
Links:
- link gunsight_link: geometry visual cylinder length=20.0 radius=0.15
Joints:
- joint gunsight_joint: origin xyz=7.5 0 0 rpy=0 1.571 0 -> xyz=10.0 0 0 rpy=0 1.571 0
